Commit message: lab3

File: src/my_r2d2/urdf/r2d2.urdf (robot description, URDF)
Before this commit: robot visual, 15 links, 14 joints
Links:
- added link base_footprint
Joints:
- added joint base_footprint_base_link_joint: type fixed, parent base_footprint, child base_link, origin xyz=0.00 0.00 0.47 rpy=0 0 0
